Commit message: change file location of 3d file

File: cheetah_description/urdf/robot_with_kinect.urdf (robot description, URDF)
Before this commit: robot yobotics, 20 links, 19 joints
Links:
- link FL_calf: geometry collision mesh filename=package://cheetah_description/meshes/calf.STL scale=1 1 1; visual mesh filename=package://cheetah_description/meshes/calf.STL scale=1 1 1
- link FL_foot: geometry collision mesh filename=package://cheetah_description/meshes/foot.STL scale=1 1 1; visual mesh filename=package://cheetah_description/meshes/foot.STL scale=1 1 1
- link FL_hip: geometry collision mesh filename=package://cheetah_description/meshes/hip.STL scale=1 1 1; visual mesh filename=package://cheetah_description/meshes/hip.STL scale=1 1 1
- link FL_thigh: geometry collision mesh filename=package://cheetah_description/meshes/thigh.STL scale=1 1 1; visual mesh filename=package://cheetah_description/meshes/thigh.STL scale=1 1 1
- link FR_calf: geometry collision mesh filename=package://cheetah_description/meshes/calf.STL scale=1 1 1; visual mesh filename=package://cheetah_description/meshes/calf.STL scale=1 1 1
- link FR_foot: geometry collision mesh filename=package://cheetah_description/meshes/foot.STL scale=1 1 1; visual mesh filename=package://cheetah_description/meshes/foot.STL scale=1 1 1
- link FR_hip: geometry collision mesh filename=package://cheetah_description/meshes/hip.STL scale=1 1 1; visual mesh filename=package://cheetah_description/meshes/hip.STL scale=1 1 1
- link FR_thigh: geometry collision mesh filename=package://cheetah_description/meshes/thigh.STL scale=1 1 1; visual mesh filename=package://cheetah_description/meshes/thigh.STL scale=1 1 1
- link RL_calf: geometry collision mesh filename=package://cheetah_description/meshes/calf.STL scale=1 1 1; visual mesh filename=file:///home/andy1/QRB_ws/install/cheetah_description/share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 scale=1 1 1
- link RL_foot: geometry collision mesh filename=package://cheetah_description/meshes/foot.STL scale=1 1 1; visual mesh filename=file:///home/andy1/QRB_ws/install/cheetah_description/share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 scale=1 1 1
- link RL_hip: geometry collision mesh filename=package://cheetah_description/meshes/hip.STL scale=1 1 1; visual mesh filename=file:///home/andy1/QRB_ws/install/cheetah_description/share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 scale=1 1 1
- link RL_thigh: geometry collision mesh filename=package://cheetah_description/meshes/thigh.STL scale=1 1 1; visual mesh filename=file:///home/andy1/QRB_ws/install/cheetah_description/share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 scale=1 1 1
- link RR_calf: geometry collision mesh filename=package://cheetah_description/meshes/calf.STL scale=1 1 1; visual mesh filename=package://cheetah_description/meshes/calf.STL scale=1 1 1
- link RR_foot: geometry collision mesh filename=package://cheetah_description/meshes/foot.STL scale=1 1 1; visual mesh filename=package://cheetah_description/meshes/foot.STL scale=1 1 1
- link RR_hip: geometry collision mesh filename=package://cheetah_description/meshes/hip.STL scale=1 1 1; visual mesh filename=package://cheetah_description/meshes/hip.STL scale=1 1 1
- link RR_thigh: geometry collision mesh filename=package://cheetah_description/meshes/thigh.STL scale=1 1 1; visual mesh filename=package://cheetah_description/meshes/thigh.STL scale=1 1 1
- link trunk: geometry collision mesh filename=package://cheetah_description/meshes/trunk.STL scale=1 1 1; visual mesh filename=file:///home/andy1/QRB_ws/install/cheetah_description/share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 scale=1 1 1

File: cheetah_description/urdf/yobotics.urdf (robot description, URDF)
Before this commit: robot yobotics_description, 25 links, 24 joints
Links:
- link FL_calf: geometry collision box size=0.016 0.016 0.2; visual mesh filename=package://cheetah_description/meshes/calf.STL scale=1 1 1
- link FL_foot: geometry collision sphere radius=0.025; visual mesh filename=package://cheetah_description/meshes/foot.STL scale=1 1 1
- link FL_hip: geometry collision box size=0.09 0.08 0.093; visual mesh filename=package://cheetah_description/meshes/hip.STL scale=1 1 1
- link FL_thigh: geometry collision box size=0.043 0.034 0.22; visual mesh filename=package://cheetah_description/meshes/thigh.STL scale=1 1 1
- link FR_calf: geometry collision box size=0.016 0.016 0.2; visual mesh filename=package://cheetah_description/meshes/calf.STL scale=1 1 1
- link FR_foot: geometry collision sphere radius=0.025; visual mesh filename=package://cheetah_description/meshes/foot.STL scale=1 1 1
- link FR_hip: geometry collision box size=0.09 0.08 0.093; visual mesh filename=package://cheetah_description/meshes/hip.STL scale=1 1 1
- link FR_thigh: geometry collision box size=0.043 0.034 0.22; visual mesh filename=package://cheetah_description/meshes/thigh.STL scale=1 1 1
- link RL_calf: geometry collision box size=0.016 0.016 0.2; visual mesh filename=file:///home/andy1/QRB_ws/install/cheetah_description/share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 scale=1 1 1
- link RL_foot: geometry collision sphere radius=0.025; visual mesh filename=file:///home/andy1/QRB_ws/install/cheetah_description/share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 scale=1 1 1
- link RL_hip: geometry collision box size=0.09 0.08 0.093; visual mesh filename=file:///home/andy1/QRB_ws/install/cheetah_description/share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 scale=1 1 1
- link RL_thigh: geometry collision box size=0.043 0.034 0.22; visual mesh filename=file:///home/andy1/QRB_ws/install/cheetah_description/share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 scale=1 1 1
- link RR_calf: geometry collision box size=0.016 0.016 0.2; visual mesh filename=package://cheetah_description/meshes/calf.STL scale=1 1 1
- link RR_foot: geometry collision sphere radius=0.025; visual mesh filename=package://cheetah_description/meshes/foot.STL scale=1 1 1
- link RR_hip: geometry collision box size=0.09 0.08 0.093; visual mesh filename=package://cheetah_description/meshes/hip.STL scale=1 1 1
- link RR_thigh: geometry collision box size=0.043 0.034 0.22; visual mesh filename=package://cheetah_description/meshes/thigh.STL scale=1 1 1
- link trunk_interia: geometry collision box size=0.3 0.2 0.093; visual mesh filename=file:///home/andy1/QRB_ws/install/cheetah_description/share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 scale=1 1 1

File: cheetah_description/xacro/leg.xacro (robot description, xacro)
@@ -1,5 +1,5 @@
 <?xml version="1.0"?>
 <robot xmlns:xacro="http://www.ros.org/wiki/xacro">
-    <xacro:include filename="$(find yobotics_description)/xacro/transmission.xacro"/>
+    <xacro:include filename="$(find cheetah_description)/xacro/transmission.xacro"/>
     <xacro:macro name="leg" params="name mirror mirror_dae front_hind front_hind_dae *origin">
 <!-- //////////////////////hip//////////////////// -->
@@ -33,5 +33,5 @@
                 </xacro:if>
                 <geometry>
-                    <mesh filename="package://yobotics_description/meshes/hip.STL" scale="1 1 1"/>
+                    <mesh filename="package://cheetah_description/meshes/hip.STL" scale="1 1 1"/>
                 </geometry>
                 <material name="gold"/>
@@ -52,5 +52,5 @@
                 </xacro:if> -->
                 <geometry>
-                    <!-- <mesh filename="package://yobotics_description/meshes/hip.STL" scale="1 1 1"/> -->
+                    <!-- <mesh filename="package://cheetah_description/meshes/hip.STL" scale="1 1 1"/> -->
                     <box size="${hip_length} ${hip_width} ${hip_height}"/>
                 </geometry>
@@ -83,5 +83,5 @@
                 </xacro:if>
                 <geometry>
-                    <mesh filename="package://yobotics_description/meshes/thigh.STL" scale="1 1 1"/>
+                    <mesh filename="package://cheetah_description/meshes/thigh.STL" scale="1 1 1"/>
                 </geometry>
                 <material name="white_blue"/>
@@ -97,5 +97,5 @@
                 <geometry>
                     <box size="${thigh_length} ${thigh_width} ${thigh_height}"/>
-                    <!-- <mesh filename="package://yobotics_description/meshes/thigh.STL" scale="1 1 1"/> -->
+                    <!-- <mesh filename="package://cheetah_description/meshes/thigh.STL" scale="1 1 1"/> -->
                 </geometry>
                 <material name="white_blue"/>
@@ -124,5 +124,5 @@
                 <origin rpy="0 0 0" xyz="0.0 0.009 0.0" />
                 <geometry>
-                    <mesh filename="package://yobotics_description/meshes/calf.STL" scale="1 1 1"/>
+                    <mesh filename="package://cheetah_description/meshes/calf.STL" scale="1 1 1"/>
                 </geometry>
                 <material name="white_blue"/>
@@ -132,5 +132,5 @@
                 <geometry>
                     <box size="${calf_length} ${calf_width} ${calf_height}"/>
-                    <!-- <mesh filename="package://yobotics_description/meshes/calf.STL" scale="1 1 1"/> -->
+                    <!-- <mesh filename="package://cheetah_description/meshes/calf.STL" scale="1 1 1"/> -->
                 </geometry>
             </collision>
@@ -153,5 +153,5 @@
                 <origin rpy="0 0 0" xyz="0 0.018 0.02"/>
                 <geometry>
-                     <mesh filename="package://yobotics_description/meshes/foot.STL" scale="1 1 1"/>
+                     <mesh filename="package://cheetah_description/meshes/foot.STL" scale="1 1 1"/>
                 </geometry>
                 <material name="white_black"/>
@@ -160,5 +160,5 @@
                 <origin rpy="0 0 0" xyz="0 0.0 0.025"/>
                 <geometry>
-                    <!-- <mesh filename="package://yobotics_description/meshes/foot.STL" scale="1 1 1"/> -->
+                    <!-- <mesh filename="package://cheetah_description/meshes/foot.STL" scale="1 1 1"/> -->
                     <sphere radius="0.025"/>
                 </geometry>

File: cheetah_description/xacro/robot.xacro (robot description, xacro)
@@ -1,8 +1,8 @@
 <?xml version="1.0"?>
 <robot name="yobotics_description" xmlns:xacro="http://www.ros.org/wiki/xacro">
-    <xacro:include filename="$(find yobotics_description)/xacro/const.xacro"/>
-    <xacro:include filename="$(find yobotics_description)/xacro/materials.xacro"/>
-    <xacro:include filename="$(find yobotics_description)/xacro/leg.xacro"/>
-    <xacro:include filename="$(find yobotics_description)/xacro/gazebo.xacro"/>
+    <xacro:include filename="$(find cheetah_description)/xacro/const.xacro"/>
+    <xacro:include filename="$(find cheetah_description)/xacro/materials.xacro"/>
+    <xacro:include filename="$(find cheetah_description)/xacro/leg.xacro"/>
+    <xacro:include filename="$(find cheetah_description)/xacro/gazebo.xacro"/>
     <!-- Debug mode will hung up the robot, use "true" or "false" to switch it. -->
     <!-- <link name="base_link">
@@ -23,7 +23,7 @@
         <visual>
             <origin rpy="0 0 0" xyz="0 0 0"/>
-            <geometry>
-                <mesh filename="package://yobotics_description/meshes/trunk.STL" scale="1 1 1"/>
-            </geometry>
+                <geometry>
+                    <mesh filename="package://cheetah_description/meshes/trunk.STL" scale="1 1 1"/>
+                </geometry>
             <material name="white_gray"/>
         </visual>
@@ -31,5 +31,5 @@
             <origin rpy="0 0 0" xyz="0 0 0"/>
             <geometry>
-               <!-- <mesh filename="package://yobotics_description/meshes/trunk.STL" scale="1 1 1"/> -->
+               <!-- <mesh filename="package://cheetah_description/meshes/trunk.STL" scale="1 1 1"/> -->
                <box size="${trunk_length} ${trunk_width} ${trunk_height}"/>
             </geometry>
@@ -87,4 +87,4 @@
         <origin rpy="0 0 0" xyz="${-leg_offset_x} ${leg_offset_y} 0"/>
     </xacro:leg>
-    <xacro:include filename="$(find yobotics_description)/xacro/accessories.urdf.xacro" />
+    <xacro:include filename="$(find cheetah_description)/xacro/accessories.urdf.xacro" />
 </robot>

File: cheetah_description/xacro/robot_with_kinect.xacro (robot description, xacro)
@@ -1,6 +1,6 @@
 <?xml version="1.0"?>
 <robot name="yobotics" xmlns:xacro="http://www.ros.org/wiki/xacro">
-	<xacro:include filename="$(find yobotics_description)/xacro/robot.xacro"/>
-	<xacro:include filename="$(find yobotics_description)/xacro/kinect.xacro" />
+	<xacro:include filename="$(find cheetah_description)/xacro/robot.xacro"/>
+	<xacro:include filename="$(find cheetah_description)/xacro/kinect.xacro" />
 	<!-- <xacro:property name="kinect_offset_x" value="0.12" /> -->
 	<xacro:property name="kinect_offset_x" value="0.25" />
